File: boardstorm_x3.kicad_sch (KiCad schematic)
At the start: 40 parts, among them J1 USB_C_Receptacle_USB2.0_14P, J2 Conn_01x20_Pin, J3 Conn_01x20_Pin, J4 Conn_01x03_Pin, SW1 SW_Push, U1 RP2040, U2 MCP1700x-330xxTT, U3 W25Q16JVSS, U4 BQ24075RGT, Y1 12 MHz

Commit message: added decoupling capacitors & voltage regulator
Parts:
- added C19: 10uF, symbol Device:C
Connections:
- net +3V3: now also C19.1
- net GND: now also C19.2
Changed lines of the file:
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@@
 	)
 	(junction
+		(at 218.44 33.02)
+		(diameter 0)
+		(color 0 0 0 0)
+	)
+	(junction
 		(at 228.6 57.15)
 		(diameter 0)
@@
 	)
 	(junction
+		(at 204.47 44.45)
+		(diameter 0)
+		(color 0 0 0 0)
+	)
+	(junction
 		(at 33.02 127)
 		(diameter 0)
@@
 	)
 	(junction
-		(at 201.93 71.12)
-		(diameter 0)
-		(color 0 0 0 0)
-	)
-	(junction
 		(at 111.76 180.34)
 		(diameter 0)
@@
 	(wire
 		(pts
+			(xy 218.44 44.45) (xy 218.44 41.91)
+		)
+		(stroke
+			(width 0)
+			(type default)
+		)
+	)
+	(wire
+		(pts
+			(xy 218.44 33.02) (xy 218.44 34.29)
+		)
+		(stroke
+			(width 0)
+			(type default)
+		)
+	)
+	(wire
+		(pts
 			(xy 214.63 87.63) (xy 205.74 87.63)
 		)
@@
 	(wire
 		(pts
-			(xy 204.47 40.64) (xy 204.47 44.45)
-		)
-		(stroke
-			(width 0)
-			(type default)
-		)
-	)
-	(wire
-		(pts
 			(xy 168.91 60.96) (xy 165.1 60.96)
 		)
@@
 	(wire
 		(pts
+			(xy 204.47 44.45) (xy 218.44 44.45)
+		)
+		(stroke
+			(width 0)
+			(type default)
+		)
+	)
+	(wire
+		(pts
 			(xy 212.09 119.38) (xy 212.09 123.19)
 		)
@@
 	(wire
 		(pts
-			(xy 204.47 71.12) (xy 201.93 71.12)
+			(xy 193.04 71.12) (xy 204.47 71.12)
 		)
 		(stroke
@@
 	(wire
 		(pts
+			(xy 204.47 40.64) (xy 204.47 44.45)
+		)
+		(stroke
+			(width 0)
+			(type default)
+		)
+	)
+	(wire
+		(pts
 			(xy 63.5 27.94) (xy 57.15 27.94)
 		)
@@
 	(wire
 		(pts
-			(xy 193.04 71.12) (xy 201.93 71.12)
-		)
-		(stroke
-			(width 0)
-			(type default)
-		)
-	)
-	(wire
-		(pts
 			(xy 60.96 43.18) (xy 60.96 30.48)
 		)
@@
 	(symbol
 		(lib_id "power:GND")
-		(at 201.93 71.12 0)
+		(at 204.47 71.12 0)
 		(unit 1)
 		(body_style 1)
@@
 		(fields_autoplaced yes)
 		(property "Reference" "#PWR030"
-			(at 201.93 77.47 0)
+			(at 204.47 77.47 0)
 			(hide yes)
 			(show_name no)
@@
 		)
 		(property "Value" "GND"
-			(at 201.93 76.2 0)
+			(at 204.47 76.2 0)
 			(show_name no)
 			(do_not_autoplace no)
@@
 		)
 		(property "Footprint" ""
-			(at 201.93 71.12 0)
+			(at 204.47 71.12 0)
 			(hide yes)
 			(show_name no)
@@
 		)
 		(property "Datasheet" ""
-			(at 201.93 71.12 0)
+			(at 204.47 71.12 0)
 			(hide yes)
 			(show_name no)
@@
 		)
 		(property "Description" "Power symbol creates a global label with name \"GND\" , ground"
-			(at 201.93 71.12 0)
+			(at 204.47 71.12 0)
 			(hide yes)
 			(show_name no)
@@
 					(unit 1)
 				)
+			)
+		)
+	)
+	(symbol
+		(lib_id "Device:C")
+		(at 218.44 38.1 0)
+		(unit 1)
+		(body_style 1)
+		(exclude_from_sim no)
+		(in_bom yes)
+		(on_board yes)
+		(in_pos_files yes)
+		(dnp no)
+		(property "Reference" "C19"
+			(at 220.726 35.56 0)
+			(show_name no)
+			(do_not_autoplace no)
+			(effects
+				(font
+					(size 1.27 1.27)
+				)
+			)
+		)
+		(property "Value" "10uF"
+			(at 221.234 40.64 0)
+			(show_name no)
+			(do_not_autoplace no)
+			(effects
+				(font
+					(size 1.27 1.27)
+				)
+			)
+		)
+		(property "Footprint" ""
+			(at 219.4052 41.91 0)
+			(hide yes)
+			(show_name no)
+			(do_not_autoplace no)
+			(effects
+				(font
+					(size 1.27 1.27)
+				)
+			)
+		)
+		(property "Datasheet" ""
+			(at 218.44 38.1 0)
+			(hide yes)
+			(show_name no)
+			(do_not_autoplace no)
+			(effects
+				(font
+					(size 1.27 1.27)
+				)
+			)
+		)
+		(property "Description" "Unpolarized capacitor"
+			(at 218.44 38.1 0)
+			(hide yes)
+			(show_name no)
+			(do_not_autoplace no)
+			(effects
+				(font
+					(size 1.27 1.27)
+				)
+			)
+		)
+		(pin "1"
+		)
+		(pin "2"
+		)
+		(instances
+			(project "boardstorm_x3"
+				(path "/ddf421bf-b812-4a1e-a1dd-65bc18fc626a"
+					(reference "C19")
+					(unit 1)
+				)
